Commit message: Added Podi's handle

File: description/urdf/pioneer3dx.urdf (robot description, URDF)
Before this commit: robot pioneer3dx, 11 links, 10 joints
Links:
- added link handle_back_plate; visual box size=0.14 0.155 0.005
- added link handle_base; visual cylinder length=0.04 radius=0.06
- added link handle_bottom; visual box size=0.33 0.155 0.035
- added link handle_bottom_plate; visual box size=0.09 0.21 0.005
- added link handle_top; visual box size=0.043 0.155 0.035
Joints:
- added joint handle_back_plate_to_bottom: type fixed, parent handle_back_plate, child handle_bottom, origin xyz=-0.14 0 0.005 rpy=0 0 0
- added joint handle_base_joint: type fixed, parent base_link, child handle_base, origin xyz=-0.13 0 0.234 rpy=0 0 0
- added joint handle_bottom_plate_to_back_plate: type fixed, parent handle_bottom_plate, child handle_back_plate, origin xyz=0.045 0 0.005 rpy=0 0.785398 0
- added joint handle_length: type prismatic, parent handle_bottom, child handle_top, origin xyz=-0.33 0 0.0275 rpy=0 0 0, axis -1 0 0, limit lower=0 upper=0.46 effort=0 velocity=1
- added joint handle_rotation: type revolute, parent handle_base, child handle_bottom_plate, origin xyz=0 0 0.04 rpy=0 0 0, axis 0 0 1, limit lower=-1.57 upper=1.57 effort=0 velocity=1

File: description/urdf/pioneer3dx.urdf.xacro (robot description, xacro)
@@ -294,6 +294,91 @@
 		<material value="Gazebo/Black"/>
 	</gazebo>
+	<!-- Zhi's Addition of Podi's handle-->
+	<link name="handle_base">
+		<visual>
+			<origin xyz="0 0 0.02" rpy="0 0 0"/>
+			<geometry>
+				<cylinder radius="0.06" length="0.04"/>
+			</geometry>
+			<material name="handleBaseBlack">
+				<color rgba="1 1 1 1"/>
+			</material>
+		</visual>
+	</link>
+	<link name="handle_bottom_plate">
+		<visual>
+			<origin xyz="0 0 0" rpy="0 0 0"/>
+			<geometry>
+				<box size="0.09 0.21 0.005" />
+			</geometry>
+			<material name="handleBottomBlack">
+				<color rgba="1 1 1 1"/>
+			</material>
+		</visual>
+	</link>
+	<link name="handle_back_plate">
+		<visual>
+			<origin xyz="-0.07 0 0" rpy="0 0 0"/>
+			<geometry>
+				<box size="0.14 0.155 0.005" />
+			</geometry>
+			<material name="handleBackPlateBlack">
+				<color rgba="1 1 1 1"/>
+			</material>
+		</visual>
+	</link>
+	<link name="handle_bottom">
+		<visual>
+			<origin xyz="-0.16666 0 0.0175" rpy="0 0 0"/>
+			<geometry>handle_rotation
+				<box size="0.33 0.155 0.035" />
+			</geometry>
+			<material name="handleBackPlateBlack">
+				<color rgba="0 0 0 1"/>
+			</material>
+		</visual>
+	</link>
+	<link name="handle_top">
+		<visual>
+			<origin xyz="-0.0215 0 -0.0175" rpy="0 0 0"/>
+			<geometry>
+				<box size="0.043 0.155 0.035" />
+			</geometry>
+			<material name="handleBackPlateBlack">
+				<color rgba="0 0 0 1"/>
+			</material>
+		</visual>
+	</link>
+	<joint name="handle_base_joint" type="fixed">
+		<origin xyz="-0.13 0 0.234" rpy="0 0 0"/>
+		<parent link="base_link"/>
+		<child link="handle_base"/>
+	</joint>
+	<joint name="handle_rotation" type="revolute">
+		<origin xyz="0 0 0.04" rpy="0 0 0"/>
+		<axis xyz = "0 0 1" />
+		<parent link="handle_base"/>
+		<child link="handle_bottom_plate"/>
+		<limit lower="-1.57" upper="1.57" effort="0" velocity="1" />
+	</joint>
+	<joint name="handle_bottom_plate_to_back_plate" type="fixed">
+		<origin xyz="0.045 0 0.005" rpy="0 0.785398 0"/>
+		<parent link="handle_bottom_plate"/>
+		<child link="handle_back_plate"/>
+	</joint>
+	<joint name="handle_back_plate_to_bottom" type="fixed">
+		<origin xyz="-0.14 0 0.005" rpy="0 0 0"/>
+		<parent link="handle_back_plate"/>
+		<child link="handle_bottom"/>
+	</joint>
+	<joint name="handle_length" type="prismatic">
+		<origin xyz="-0.33 0 0.0275" rpy="0 0 0"/>
+		<axis xyz ="-1 0 0" />
+		<parent link="handle_bottom"/>
+		<child link="handle_top"/>
+		<limit lower="0" upper="0.46" effort="0" velocity="1" />
+	</joint>
 	<create>
-	<back_sonar parent="base_link"/>
+	<!-- <back_sonar parent="base_link"/> -->
   	<top_plate  parent="base_link"/>
   	</create>
